Commit message: robot model updated

File: src/mob_description/urdf/common_properties.xacro (robot description, xacro)
@@ -40,11 +40,45 @@
     <visual>
         <geometry>
-            <box size="0.1 0.1 0.1" />
+            <box size="0.015 0.040 0.030" />
         </geometry>
+        <material name="${color}" />
         <origin xyz="0 0 0" rpy="0 0 0" />
-        <material name="${color}" />
     </visual>
-  <mass value = "0.1" />
-    <inertia ixx="0.000166667" iyy = "0.000166667" izz="0.000166667" />
+    <visual>
+        <geometry>
+            <cylinder radius="0.010" length="0.015"/>
+        </geometry>
+        <material name="green" />
+        <origin xyz="0.0075 0 0" rpy="0 ${pi / 2.0} 0" />
+    </visual>
+    <mass value = "0.1" />
+        <inertia ixx="0.000166667" iyy = "0.000166667" izz="0.000166667" />
+    </xacro:macro>
+   <xacro:macro name="wheel_link" params="prefix">
+        <link name="${prefix}_wheel_link">
+            <visual>
+                <geometry>
+                    <cylinder radius="${wheel_radius}" length="${wheel_length}" />
+                </geometry>
+                <origin xyz="0 0 0" rpy="${pi / 2.0} 0 0" />
+                <material name="gray" />
+            </visual>
+            <collision>
+                <geometry>
+                    <sphere radius="${wheel_radius}" />
+                </geometry>
+                <origin xyz="0 0 0" rpy="0 0 0" />
+            </collision>
+            <xacro:cylinder_inertia m="1.0" r="${wheel_radius}" l="${wheel_length}"
+                                    o_xyz="0 0 0" o_rpy="${pi / 2.0} 0 0" />
+        </link>
+    </xacro:macro>
+    <xacro:macro name = "wheel_joint" params = "child_prefix xyz">
+        <joint name="base_${child_prefix}_wheel_joint" type="continuous">
+            <parent link="base_link" />
+            <child link="${child_prefix}_wheel_link" />
+            <origin xyz="${xyz}" rpy="0 0 0" />
+            <axis xyz="0 1 0" />
+        </joint>
     </xacro:macro>
 </robot>

File: src/mob_description/urdf/mobile_base.xacro (robot description, xacro)
@@ -1,9 +1,9 @@
 <?xml version="1.0"?>
 <robot xmlns:xacro="http://www.ros.org/wiki/xacro">
-    <xacro:property name="base_length" value="0.6" />
-    <xacro:property name="base_width" value="0.4" />
-    <xacro:property name="base_height" value="0.2" />
-    <xacro:property name="wheel_radius" value="0.1" />
-    <xacro:property name="wheel_length" value="0.05" />
+    <xacro:property name="base_length" value="0.312" />
+    <xacro:property name="base_width" value="0.2115" />
+    <xacro:property name="base_height" value="0.002" />
+    <xacro:property name="wheel_radius" value="0.0325" />
+    <xacro:property name="wheel_length" value="0.025" />
     <link name="base_footprint" />
     <link name="base_link">
@@ -24,42 +24,8 @@
                            o_xyz="0 0 ${base_height / 2.0}" o_rpy="0 0 0" />
     </link>
-    <xacro:macro name="wheel_link" params="prefix">
-        <link name="${prefix}_wheel_link">
-            <visual>
-                <geometry>
-                    <cylinder radius="${wheel_radius}" length="${wheel_length}" />
-                </geometry>
-                <origin xyz="0 0 0" rpy="${pi / 2.0} 0 0" />
-                <material name="gray" />
-            </visual>
-            <collision>
-                <geometry>
-                    <sphere radius="${wheel_radius}" />
-                </geometry>
-                <origin xyz="0 0 0" rpy="0 0 0" />
-            </collision>
-            <xacro:cylinder_inertia m="1.0" r="${wheel_radius}" l="${wheel_length}"
-                                    o_xyz="0 0 0" o_rpy="${pi / 2.0} 0 0" />
-        </link>
-    </xacro:macro>
-    <xacro:wheel_link prefix="right" />
-    <xacro:wheel_link prefix="left" />
-    <link name="caster_wheel_link">
-        <visual>
-            <geometry>
-                <sphere radius="${wheel_radius / 2.0}" />
-            </geometry>
-            <origin xyz="0 0 0" rpy="0 0 0" />
-            <material name="gray" />
-        </visual>
-        <collision>
-            <geometry>
-                <sphere radius="${wheel_radius / 2.0}" />
-            </geometry>
-            <origin xyz="0 0 0" rpy="0 0 0" />
-        </collision>
-        <xacro:sphere_inertia m="0.5" r="${wheel_radius / 2.0}"
-                              o_xyz="0 0 0" o_rpy="0 0 0" />
-    </link>
+    <xacro:wheel_link prefix="right_back" />
+    <xacro:wheel_link prefix="left_back" />
+    <xacro:wheel_link prefix="right_front" />
+    <xacro:wheel_link prefix="left_front" />
     <link name="camera_link">
         <xacro:camera width="640" height="480" hfov="1.3962634" color="black" />
@@ -70,25 +36,12 @@
         <origin xyz="0 0 ${wheel_radius}" rpy="0 0 0" />
     </joint>
-    <joint name="base_right_wheel_joint" type="continuous">
-        <parent link="base_link" />
-        <child link="right_wheel_link" />
-        <origin xyz="${-base_length / 4.0} ${-(base_width + wheel_length) / 2.0} 0" rpy="0 0 0" />
-        <axis xyz="0 1 0" />
-    </joint>
-    <joint name="base_left_wheel_joint" type="continuous">
-        <parent link="base_link" />
-        <child link="left_wheel_link" />
-        <origin xyz="${-base_length / 4.0} ${(base_width + wheel_length) / 2.0} 0" rpy="0 0 0" />
-        <axis xyz="0 1 0" />
-    </joint>
-    <joint name="base_caster_wheel_joint" type="fixed">
-        <parent link="base_link" />
-        <child link="caster_wheel_link" />
-        <origin xyz="${base_length / 3.0} 0 ${-wheel_radius / 2.0}" rpy="0 0 0" />
-    </joint>
+    <xacro:wheel_joint child_prefix = "right_back" xyz = "${(-base_length / 2.0)+0.012} ${-(base_width + wheel_length) / 2.0} -0.020"/>
+    <xacro:wheel_joint child_prefix = "left_back" xyz = "${(-base_length / 2.0)+0.012} ${(base_width + wheel_length) / 2.0} -0.020"/>
+    <xacro:wheel_joint child_prefix = "left_front" xyz = "${(base_length / 2.0)-0.012} ${-(base_width + wheel_length) / 2.0} -0.020"/>
+    <xacro:wheel_joint child_prefix = "right_front" xyz = "${(base_length / 2.0)-0.012} ${(base_width + wheel_length) / 2.0} -0.020"/>
     <joint name="base_camera_joint" type="fixed">
         <parent link="base_link"/>
         <child link="camera_link"/>
-        <origin xyz="${base_length/2+0.05} 0.0 ${wheel_radius + base_height - 0.2}" rpy="0.0 0.0 0.0"/>
+        <origin xyz="${base_length/2 - 0.050} 0.0 ${base_height+0.015}" rpy="0.0 0.0 0.0"/>
         <!-- <limit lower="0.0" upper="180.0" effort="0.0" velocity="1.0"/> -->
     </joint>

File: src/mob_description/urdf/mobile_base_gazebo.xacro (robot description, xacro)
@@ -46,16 +46,16 @@
     </gazebo>
     <gazebo reference="camera_link">
-    <sensor name="imu_sensor" type="imu">
-    <always_on>1</always_on>
-    <update_rate>1</update_rate>
-    <visualize>true</visualize>
-    <topic>imu</topic>
-</sensor>
-</gazebo>
-    <gazebo>
-        <plugin
-            filename="gz-sim-joint-state-publisher-system"
-            name="gz::sim::systems::JointStatePublisher">
-        </plugin>
-   </gazebo>
+      <sensor name="imu_sensor" type="imu">
+      <always_on>1</always_on>
+      <update_rate>1</update_rate>
+      <visualize>true</visualize>
+      <topic>imu</topic>
+      </sensor>
+  </gazebo>
+  <gazebo>
+      <plugin
+          filename="gz-sim-joint-state-publisher-system"
+          name="gz::sim::systems::JointStatePublisher">
+      </plugin>
+  </gazebo>
 </robot>

Commit message: Camera testing added

File: src/mob_description/urdf/common_properties.xacro (robot description, xacro)
@@ -74,10 +74,10 @@
         </link>
     </xacro:macro>
-    <xacro:macro name = "wheel_joint" params = "child_prefix xyz">
+    <xacro:macro name = "wheel_joint" params = "child_prefix xyz xyz_axis">
         <joint name="base_${child_prefix}_wheel_joint" type="continuous">
             <parent link="base_link" />
             <child link="${child_prefix}_wheel_link" />
             <origin xyz="${xyz}" rpy="0 0 0" />
-            <axis xyz="0 1 0" />
+            <axis xyz="${xyz_axis}" />
         </joint>
     </xacro:macro>

File: src/mob_description/urdf/mobile_base.xacro (robot description, xacro)
@@ -34,10 +34,10 @@
         <parent link="base_footprint" />
         <child link="base_link" />
-        <origin xyz="0 0 ${wheel_radius}" rpy="0 0 0" />
+        <origin xyz="0 0 ${wheel_radius+0.012}" rpy="0 0 0" />
     </joint>
-    <xacro:wheel_joint child_prefix = "right_back" xyz = "${(-base_length / 2.0)+0.012} ${-(base_width + wheel_length) / 2.0} -0.020"/>
-    <xacro:wheel_joint child_prefix = "left_back" xyz = "${(-base_length / 2.0)+0.012} ${(base_width + wheel_length) / 2.0} -0.020"/>
-    <xacro:wheel_joint child_prefix = "left_front" xyz = "${(base_length / 2.0)-0.012} ${-(base_width + wheel_length) / 2.0} -0.020"/>
-    <xacro:wheel_joint child_prefix = "right_front" xyz = "${(base_length / 2.0)-0.012} ${(base_width + wheel_length) / 2.0} -0.020"/>
+    <xacro:wheel_joint child_prefix = "right_back" xyz = "${(-base_length / 2.0)+0.012} ${-(base_width + wheel_length) / 2.0} -0.020" xyz_axis = "0 1 0"/>
+    <xacro:wheel_joint child_prefix = "left_back" xyz = "${(-base_length / 2.0)+0.012} ${(base_width + wheel_length) / 2.0} -0.020" xyz_axis = "0 1 0"/>
+    <xacro:wheel_joint child_prefix = "left_front" xyz = "${(base_length / 2.0)-0.012} ${-(base_width + wheel_length) / 2.0} -0.020" xyz_axis = "0 1 0"/>
+    <xacro:wheel_joint child_prefix = "right_front" xyz = "${(base_length / 2.0)-0.012} ${(base_width + wheel_length) / 2.0} -0.020" xyz_axis = "0 1 0"/>
     <joint name="base_camera_joint" type="fixed">
         <parent link="base_link"/>

File: src/mob_description/urdf/mobile_base_gazebo.xacro (robot description, xacro)
@@ -12,6 +12,6 @@
             filename="gz-sim-diff-drive-system"
             name="gz::sim::systems::DiffDrive">
-            <left_joint>base_left_wheel_joint</left_joint>
-            <right_joint>base_right_wheel_joint</right_joint>
+            <left_joint>base_left_back_wheel_joint</left_joint>
+            <right_joint>base_right_back_wheel_joint</right_joint>
             <frame_id>odom</frame_id>
             <child_frame_id>base_footprint</child_frame_id>

Commit message: Robot arm integrated

File: src/mob_description/urdf/common_properties.xacro (robot description, xacro)
@@ -4,4 +4,7 @@
         <color rgba="0 0.6 0 1" />
     </material>
+  <material name="silver">
+    <color rgba="0.8 0.8 0.8 1.0"/>
+  </material>
     <material name="gray">
         <color rgba="0.7 0.7 0.7 1" />
@@ -82,3 +85,70 @@
         </joint>
     </xacro:macro>
+<xacro:macro name="robo_link" params="name radius length material mass">
+  <link name="${name}">
+      <visual>
+        <geometry>
+          <cylinder length="${length}" radius="${radius}"/>
+        </geometry>
+          <origin xyz="0.0 0.0 ${length/2}" rpy="0.0 0.0 0.0"/>
+        <material name="${material}"/>
+      </visual>
+      <collision>
+          <geometry>
+              <cylinder length="${length}" radius="${radius}"/>
+          </geometry>
+          <origin xyz="0.0 0.0 ${length/2}" rpy="0.0 0.0 0.0"/>
+      </collision>
+      <inertial>
+          <mass value="${mass}" />
+          <origin xyz="0 0 0" rpy="0 0 0" />
+          <inertia ixx="${(mass/12) * (3*radius*radius + length*length)}" ixy="0" ixz="0"
+                  iyy="${(mass/12) * (3*radius*radius + length*length)}" iyz="0"
+                  izz="${(mass/2) * (radius*radius)}" />
+      </inertial>
+    </link>
+</xacro:macro>
+<!-- <xacro:macro name="gripper_finger" params="no side">
+  <link name="gripper_finger_${no}">
+    <visual>
+      <geometry>
+        <box size="0.01 0.03 0.03"/>
+      </geometry>
+      <origin xyz="0.005 0 0.015" rpy="0.0 0.0 0.0"/>
+      <material name="silver"/>
+    </visual>
+  </link>
+</xacro:macro> -->
+<xacro:macro name = "box_link" params = "name sx sy sz material mass">
+  <link name="${name}">
+    <visual>
+      <geometry>
+        <box size="${sx} ${sy} ${sz}"/>
+      </geometry>
+      <origin xyz="0.0 0.0 0.05" rpy="0.0 0.0 0.0"/>
+      <material name="${material}"/>
+    </visual>
+    <collision>
+      <geometry>
+        <box size="${sx} ${sy} ${sz}"/>
+      </geometry>
+      <origin xyz="0.0 0.0 0.05" rpy="0.0 0.0 0.0"/>
+    </collision>
+  <inertial>
+  <mass value="${mass}"/>
+  <origin xyz="0 0 0" rpy="0 0 0" />
+  <inertia ixx="${mass*(sy*sy + sz* sz)/12}" ixy="0.0" ixz="0.0" iyy="${mass*(sx*sx + sz* sz)/12}" iyz="0.0" izz="${mass*(sy*sy + sx* sx)/12}"/>
+  </inertial>
+  </link>
+</xacro:macro>
+<xacro:macro name="ros2_control_joint" params = "name mi ma">
+  <joint name="${name}">
+        <command_interface name = "position">
+            <param name="min" value="${mi}"/>
+            <param name="max" value="${ma}"/>
+        </command_interface>
+        <state_interface name = "velocity" />
+        <state_interface name = "position"/>
+    </joint>
+</xacro:macro>
 </robot>

File: src/mob_description/urdf/mobile_base.xacro (robot description, xacro)
@@ -46,3 +46,8 @@
         <!-- <limit lower="0.0" upper="180.0" effort="0.0" velocity="1.0"/> -->
     </joint>
+    <joint name = "robo_base_joint" type = "fixed">
+        <parent link="base_link"/>
+        <child link="base_robot_link"/>
+        <origin xyz="${base_length/2.0} 0 0" rpy="0 0 0" />
+    </joint>
 </robot>

File: src/mob_description/urdf/my_robot.urdf.xacro (robot description, xacro)
@@ -4,3 +4,4 @@
     <xacro:include filename="$(find mob_description)/urdf/common_properties.xacro" />
     <xacro:include filename="$(find mob_description)/urdf/mobile_base.xacro" />
+    <xacro:include filename="$(find mob_description)/urdf/arm_base.xacro" />
 </robot>
