Commit message: excavator mechanism added

File: src/mob_description/urdf/arm_base.xacro (robot description, xacro)
@@ -1,11 +1,9 @@
 <?xml version="1.0"?>
 <robot name="three_axis_arm" xmlns:xacro="http://ros.org/wiki/xacro">
-<xacro:robo_link name="base_robot_link" radius= "0.1" length="0.1" material="black" mass="0.2"/>
-<xacro:robo_link name="link_1" radius= "0.05" length="0.1" material="silver" mass="0.15"/>
-<xacro:robo_link name="link_2" radius= "0.04" length="0.4" material="black" mass="0.45" />
-<xacro:robo_link name="link_3" radius= "0.03" length="0.2" material="silver" mass="0.05" />
+<xacro:robo_link name="base_robot_link" radius= "0.05" length="0.03" material="black" mass="0.2"/>
+<xacro:robo_link name="link_1" radius= "0.01" length="0.03" material="silver" mass="0.15"/>
+<xacro:robo_link name="link_2" radius= "0.01" length="0.15" material="black" mass="0.45" />
+<xacro:robo_link name="link_3" radius= "0.01" length="0.15" material="silver" mass="0.05" />
 <xacro:box_link name="gripper" sx="0.05" sy="0.05" sz="0.1" material="black" mass="0.1"/>
-<xacro:box_link name = "gripper_finger_1" sx="0.01" sy="0.03" sz="0.03" material="silver" mass="0.01"/>
-<xacro:box_link name = "gripper_finger_2" sx="0.01" sy="0.03" sz="0.03" material="silver" mass="0.01"/>
   <!-- <link name="gripper">
     <visual>
@@ -48,5 +46,5 @@
     <parent link="link_1"/>
     <child link="link_2"/>
-    <origin xyz="0 -0.02 0.1" rpy="0 0 0"/>
+    <origin xyz="0 -0.02 0.025" rpy="0 0 0"/>
     <axis xyz="0 1 0"/>
     <limit lower="-1.57" upper="1.57" effort="10" velocity="1.0"/>
@@ -56,28 +54,16 @@
     <parent link="link_2"/>
     <child link="link_3"/>
-    <origin xyz="0 0.02 0.4" rpy="0 0 0"/>
+    <origin xyz="0 0.02 0.15" rpy="0 0 0"/>
     <axis xyz="0 1 0"/>
     <limit lower="-1.57" upper="1.57" effort="10" velocity="1.0"/>
   </joint>
   <!-- Gripper -->
-  <joint name="gripper_joint" type="fixed">
+  <joint name="gripper_joint" type="revolute">
     <parent link="link_3"/>
     <child link="gripper"/>
-    <origin xyz="0 0.0 0.2" rpy="0 0 0"/>
+    <origin xyz="0.0 -0.01 0.15" rpy="1.57 0.0 3.14"/>
+    <axis xyz="0 0 1"/>
+    <limit lower="-1.57" upper="1.57" effort="10" velocity="1.0"/>
   </joint>
   <!-- End Effector -->
-  <joint name="gripper_finger_1_joint" type="prismatic">
-    <parent link="gripper"/>
-    <child link="gripper_finger_1"/>
-    <origin xyz="0.005 0 0.1" rpy="0 0 0"/>
-    <axis xyz="1 0 0"/>
-    <limit lower="0" upper="0.025" effort="5" velocity="0.5"/>
-  </joint>
-  <joint name="gripper_finger_2_joint" type="prismatic">
-    <parent link="gripper"/>
-    <child link="gripper_finger_2"/>
-    <origin xyz="-0.005 0 0.1" rpy="0 0 0"/>
-    <axis xyz="-1 0 0"/>
-    <limit lower="0" upper="0.025" effort="5" velocity="0.5"/>
-  </joint>
 </robot>

File: src/mob_description/urdf/common_properties.xacro (robot description, xacro)
@@ -109,22 +109,12 @@
     </link>
 </xacro:macro>
-<!-- <xacro:macro name="gripper_finger" params="no side">
-  <link name="gripper_finger_${no}">
-    <visual>
-      <geometry>
-        <box size="0.01 0.03 0.03"/>
-      </geometry>
-      <origin xyz="0.005 0 0.015" rpy="0.0 0.0 0.0"/>
-      <material name="silver"/>
-    </visual>
-  </link>
-</xacro:macro> -->
 <xacro:macro name = "box_link" params = "name sx sy sz material mass">
   <link name="${name}">
     <visual>
       <geometry>
-        <box size="${sx} ${sy} ${sz}"/>
+      <!-- <box size="0.1 0.1 0.1"/> -->
+        <mesh filename="file://$(find mob_description)/stl/excavator.stl" scale="0.001 0.001 0.001"/>
       </geometry>
-      <origin xyz="0.0 0.0 0.05" rpy="0.0 0.0 0.0"/>
+      <origin xyz="0.0 0.0 0.0" rpy="0.0 0.0 0.0"/>
       <material name="${material}"/>
     </visual>
@@ -133,5 +123,5 @@
         <box size="${sx} ${sy} ${sz}"/>
       </geometry>
-      <origin xyz="0.0 0.0 0.05" rpy="0.0 0.0 0.0"/>
+      <origin xyz="0.0 0.0 0.0" rpy="0.0 0.0 0.0"/>
     </collision>
   <inertial>
