Commit message: robot description updated

File: mob_description/urdf/arm_base.xacro (robot description, xacro)
@@ -2,8 +2,8 @@
 <robot name="three_axis_arm" xmlns:xacro="http://ros.org/wiki/xacro">
 <xacro:robo_link name="base_robot_link" radius= "0.05" length="0.03" material="black" mass="0.2"/>
-<xacro:robo_link name="link_1" radius= "0.01" length="0.03" material="silver" mass="0.15"/>
+<xacro:robo_link name="link_1" radius= "0.01" length="0.03" material="orange" mass="0.15"/>
 <xacro:robo_link name="link_2" radius= "0.01" length="0.15" material="black" mass="0.45" />
-<xacro:robo_link name="link_3" radius= "0.01" length="0.15" material="silver" mass="0.05" />
-<xacro:box_link name="gripper" sx="0.05" sy="0.05" sz="0.1" material="black" mass="0.1"/>
+<xacro:robo_link name="link_3" radius= "0.01" length="0.15" material="orange" mass="0.05" />
+<xacro:box_link name="gripper" sx="0.05" sy="0.05" sz="0.1" material="dark_gray" mass="0.1"/>
   <!-- <link name="gripper">
     <visual>
@@ -38,5 +38,5 @@
     <parent link="base_robot_link"/>
     <child link="link_1"/>
-    <origin xyz="0 0 0.05" rpy="0 0 0"/>
+    <origin xyz="0 0 0.03" rpy="0 0 0"/>
     <axis xyz="0 0 1"/>
     <limit lower="-3.14" upper="3.14" effort="10" velocity="1.0"/>

File: mob_description/urdf/common_properties.xacro (robot description, xacro)
@@ -8,8 +8,14 @@
   </material>
     <material name="gray">
-        <color rgba="0.7 0.7 0.7 1" />
+        <color rgba="0.3 0.3 0.3 1" />
+    </material>
+    <material name="dark_gray">
+        <color rgba="0.2 0.2 0.2 1" />
     </material>
     <material name = "black">
-        <color rgba="0 0 0 1"/>
+        <color rgba="0.1 0.1 0.1 1"/>
+    </material>
+    <material name = "orange">
+        <color rgba="1.0 0.5 0.0 1"/>
     </material>
     <xacro:macro name="box_inertia" params="m x y z o_xyz o_rpy">
@@ -65,5 +71,5 @@
                 </geometry>
                 <origin xyz="0 0 0" rpy="${pi / 2.0} 0 0" />
-                <material name="gray" />
+                <material name="dark_gray" />
             </visual>
             <collision>

File: mob_description/urdf/mobile_base.xacro (robot description, xacro)
@@ -29,5 +29,5 @@
     <xacro:wheel_link prefix="left_front" />
     <link name="camera_link">
-        <xacro:camera width="640" height="480" hfov="1.3962634" color="black" />
+        <xacro:camera width="640" height="480" hfov="1.3962634" color="gray" />
     </link>
     <joint name="base_joint" type="fixed">
@@ -43,5 +43,5 @@
         <parent link="base_link"/>
         <child link="camera_link"/>
-        <origin xyz="${base_length/2 - 0.050} 0.0 ${base_height+0.015}" rpy="0.0 0.0 0.0"/>
+        <origin xyz="${base_length/2 -0.02} 0.0 ${base_height+0.015}" rpy="0.0 0.0 0.0"/>
         <!-- <limit lower="0.0" upper="180.0" effort="0.0" velocity="1.0"/> -->
     </joint>
@@ -49,5 +49,5 @@
         <parent link="base_link"/>
         <child link="base_robot_link"/>
-        <origin xyz="${base_length/2.0} 0 0" rpy="0 0 0" />
+        <origin xyz="${base_length/2.0 - 0.08} 0.0 0.002" rpy="0 0 0" />
     </joint>
 </robot>
